File: pcb/_autosave-pcb.kicad_pcb (KiCad board)
At the start: 2 copper layers, 155 parts, among them J1 AVR-ISP-6, SW1 ESCAPE, SW10 #9, SW11 #0, SW12 -_, SW13 =+, SW14 BKSPC, SW15 DELETE, SW16 TAB, SW17 Q, SW18 W, SW19 E, SW2 #1, SW20 R, SW21 T, SW22 Y, SW23 U, SW24 I, SW25 O, SW26 P, SW27 [{, SW28 ]}, SW29 \|, SW3 #2, SW30 `~, SW31 CAP, SW32 A, SW33 D, SW34 S, SW35 F, SW36 G, SW37 H, SW38 J, SW39 K, SW4 #3, SW40 L, SW41 ;:, SW42 '", SW43 ENTER, SW44 PGUP, SW45 SHIFT, SW46 Z, SW47 X, SW48 C, SW49 V, SW5 #4, SW50 B, SW51 N, SW52 M, SW53 ,<, SW54 .>, SW55 /?, SW56 SHIFT, SW57 UPROW, SW58 PGDOWN, SW59 CRTL, SW6 #5, SW60 WIN, SW61 ALT, SW62 SPACE, SW63 ALT, SW64 FN, SW65 LEFTROW, SW66 DOWNROW, SW67 RIGHTROW, SW7 #6, SW8 #7, SW9 #8, U1 PRTR5V0U2X, U2 ATmega32U4-A, Y1 Crystal_GND24_Small

Commit message: Keys and Diodes laid out
Connections:
- D1 pad 1: col0 -> row0
- D10 pad 1: col0 -> row0
- D11 pad 1: col0 -> row0
- D12 pad 1: col0 -> row0
- D13 pad 1: col0 -> row0
- D14 pad 1: col0 -> row0
- D15 pad 1: col0 -> row0
- D16 pad 1: col0 -> row1
- D17 pad 1: col0 -> row1
- D18 pad 1: col0 -> row1
- D19 pad 1: col0 -> row1
- D2 pad 1: col0 -> row0
- D20 pad 1: col0 -> row1
- D21 pad 1: col0 -> row1
- D22 pad 1: col0 -> row1
- D23 pad 1: col0 -> row1
- D24 pad 1: col0 -> row1
- D25 pad 1: col0 -> row1
- D26 pad 1: col0 -> row1
- D27 pad 1: col0 -> row1
- D28 pad 1: col0 -> row1
- D29 pad 1: col0 -> row1
- D3 pad 1: col0 -> row0
- D30 pad 1: col0 -> row1
- D31 pad 1: col0 -> col13
- D32 pad 1: col0 -> col13
- D33 pad 1: col0 -> col13
- D34 pad 1: col0 -> col13
- D35 pad 1: col0 -> col13
- D36 pad 1: col0 -> col13
- D37 pad 1: col0 -> col13
- D38 pad 1: col0 -> col13
- D39 pad 1: col0 -> col13
- D4 pad 1: col0 -> row0
- D40 pad 1: col0 -> col13
- D41 pad 1: col0 -> col13
- D42 pad 1: col0 -> col13
- D43 pad 1: col0 -> col13
- D44 pad 1: col0 -> col13
- D45 pad 1: col0 -> col11
- D46 pad 1: col0 -> col11
- D47 pad 1: col0 -> col11
- D48 pad 1: col0 -> col11
- D49 pad 1: col0 -> col11
- D5 pad 1: col0 -> row0
- D50 pad 1: col0 -> col11
- D51 pad 1: col0 -> col11
- D52 pad 1: col0 -> col11
- D53 pad 1: col0 -> col11
- D54 pad 1: col0 -> col11
- D55 pad 1: col0 -> col11
- D56 pad 1: col0 -> col11
- D57 pad 1: col0 -> col11
- D58 pad 1: col0 -> col11
- D59 pad 1: col0 -> row4
- D6 pad 1: col0 -> row0
- D60 pad 1: col0 -> row4
- D61 pad 1: col0 -> row4
- D62 pad 1: col0 -> row4
- D63 pad 1: col0 -> row4
- D64 pad 1: col0 -> row4
- D65 pad 1: col0 -> row4
- D66 pad 1: col0 -> row4
- D67 pad 1: col0 -> row4
- D7 pad 1: col0 -> row0
- D8 pad 1: col0 -> row0
- D9 pad 1: col0 -> row0
- SW10 pad 2: col0 -> col9
- SW11 pad 2: col0 -> col10
- SW12 pad 2: col0 -> col11
- SW13 pad 2: col0 -> col12
- SW14 pad 2: col0 -> col13
- SW17 pad 2: col0 -> col1
- SW18 pad 2: col0 -> col2
- SW19 pad 2: col0 -> col3
- SW2 pad 2: col0 -> col1
- SW20 pad 2: col0 -> col4
- SW21 pad 2: col0 -> col5
- SW22 pad 2: col0 -> col6
- SW23 pad 2: col0 -> col7
- SW24 pad 2: col0 -> col8
- SW25 pad 2: col0 -> col9
- SW26 pad 2: col0 -> col10
- SW27 pad 2: col0 -> col11
- SW28 pad 2: col0 -> col12
- SW29 pad 2: col0 -> col13
- SW3 pad 2: col0 -> col2
- SW32 pad 2: col0 -> col1
- SW33 pad 2: col0 -> col2
- SW34 pad 2: col0 -> col3
- SW35 pad 2: col0 -> row1
- SW36 pad 2: col0 -> col5
- SW37 pad 2: col0 -> col6
- SW38 pad 2: col0 -> col7
- SW39 pad 2: col0 -> col8
- SW4 pad 2: col0 -> col3
- SW40 pad 2: col0 -> col9
- SW41 pad 2: col0 -> col10
- SW42 pad 2: col0 -> col11
- SW43 pad 2: col0 -> col12
- SW46 pad 2: col0 -> col1
- SW47 pad 2: col0 -> col2
- SW48 pad 2: col0 -> col3
- SW49 pad 2: col0 -> row1
- SW5 pad 2: col0 -> col4
- SW50 pad 2: col0 -> col5
- SW51 pad 2: col0 -> col6
- SW52 pad 2: col0 -> col7
- SW53 pad 2: col0 -> col8
- SW54 pad 2: col0 -> col9
- SW55 pad 2: col0 -> col10
- SW56 pad 2: col0 -> col12
- SW57 pad 2: col0 -> col13
- SW6 pad 2: col0 -> col5
- SW60 pad 2: col0 -> col1
- SW61 pad 2: col0 -> col2
- SW62 pad 2: col0 -> col6
- SW63 pad 2: col0 -> col10
- SW64 pad 2: col0 -> col11
- SW65 pad 2: col0 -> col12
- SW66 pad 2: col0 -> col13
- SW7 pad 2: col0 -> col6
- SW8 pad 2: col0 -> col7
- SW9 pad 2: col0 -> col8
- U2 pad 1: col0 -> row0
- U2 pad 19: col0 -> col8
- U2 pad 20: col0 -> col9
- U2 pad 21: col0 -> col10
- U2 pad 22: col0 -> col12
- U2 pad 25: col0 -> col11
- U2 pad 26: col0 -> col13
- U2 pad 29: col0 -> col1
- U2 pad 30: col0 -> col2
- U2 pad 31: col0 -> col3
- U2 pad 32: col0 -> col4
- U2 pad 36: col0 -> col6
- U2 pad 37: col0 -> col5
- U2 pad 38: col0 -> row1
- U2 pad 39: col0 -> row4
- U2 pad 40: col0 -> col11
- U2 pad 41: col0 -> col13
- U2 pad 8: col0 -> col7
