File: pcb/matrix.kicad_sch (KiCad schematic)
At the start: 134 parts, among them SW1 ESCAPE, SW10 #9, SW11 #0, SW12 -_, SW13 =+, SW14 BKSPC, SW15 DELETE, SW16 TAB, SW17 Q, SW18 W, SW19 E, SW2 #1, SW20 R, SW21 T, SW22 Y, SW23 U, SW24 I, SW25 O, SW26 P, SW27 [{, SW28 ]}, SW29 \|, SW3 #2, SW30 `~, SW31 CAP, SW32 A, SW33 D, SW34 S, SW35 F, SW36 G, SW37 H, SW38 J, SW39 K, SW4 #3, SW40 L, SW41 ;:, SW42 '", SW43 ENTER, SW44 PGUP, SW45 SHIFT, SW46 Z, SW47 X, SW48 C, SW49 V, SW5 #4, SW50 B, SW51 N, SW52 M, SW53 ,<, SW54 .>, SW55 /?, SW56 SHIFT, SW57 UPROW, SW58 PGDOWN, SW59 CRTL, SW6 #5, SW60 WIN, SW61 ALT, SW62 SPACE, SW63 ALT, SW64 FN, SW65 LEFTROW, SW66 DOWNROW, SW67 RIGHTROW, SW7 #6, SW8 #7, SW9 #8

Commit message: Routing Finished
Connections:
- net col4: no longer D16.1 (K), D17.1 (K), D18.1 (K), D19.1 (K), D20.1 (K), D21.1 (K), D22.1 (K), D23.1 (K), D24.1 (K), D25.1 (K), D26.1 (K), D27.1 (K), D28.1 (K), D29.1 (K), D30.1 (K)
- new net row1: D16.1 (K), D17.1 (K), D18.1 (K), D19.1 (K), D20.1 (K), D21.1 (K), D22.1 (K), D23.1 (K), D24.1 (K), D25.1 (K), D26.1 (K), D27.1 (K), D28.1 (K), D29.1 (K), D30.1 (K)
Changed lines of the file:
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@@
 	)
 	(junction
-		(at 138.43 113.03)
-		(diameter 0)
-		(color 0 0 0 0)
-	)
-	(junction
 		(at 50.8 90.17)
 		(diameter 0)
@@
 	(wire
 		(pts
-			(xy 138.43 102.87) (xy 138.43 113.03)
+			(xy 138.43 102.87) (xy 138.43 125.73)
 		)
 		(stroke
@@
 	(wire
 		(pts
-			(xy 127 113.03) (xy 138.43 113.03)
+			(xy 127 113.03) (xy 146.05 113.03)
 		)
 		(stroke
@@
 	(wire
 		(pts
-			(xy 138.43 113.03) (xy 146.05 113.03)
-		)
-		(stroke
-			(width 0)
-			(type default)
-		)
-	)
-	(wire
-		(pts
 			(xy 328.93 102.87) (xy 328.93 125.73)
 		)
@@
 		)
 		(stroke
-			(width 0)
-			(type default)
-		)
-	)
-	(wire
-		(pts
-			(xy 138.43 113.03) (xy 138.43 125.73)
-		)
-		(stroke
