File: pcb/pcb.kicad_pcb (KiCad board)
At the start: 2 copper layers, 305 x 104.8 mm, 155 parts, among them J1 AVR-ISP-6, SW1 ESCAPE, SW10 #9, SW11 #0, SW12 -_, SW13 =+, SW14 BKSPC, SW15 DELETE, SW16 TAB, SW17 Q, SW18 W, SW19 E, SW2 #1, SW20 R, SW21 T, SW22 Y, SW23 U, SW24 I, SW25 O, SW26 P, SW27 [{, SW28 ]}, SW29 \|, SW3 #2, SW30 `~, SW31 CAP, SW32 A, SW33 D, SW34 S, SW35 F, SW36 G, SW37 H, SW38 J, SW39 K, SW4 #3, SW40 L, SW41 ;:, SW42 '", SW43 ENTER, SW44 PGUP, SW45 SHIFT, SW46 Z, SW47 X, SW48 C, SW49 V, SW5 #4, SW50 B, SW51 N, SW52 M, SW53 ,<, SW54 .>, SW55 /?, SW56 SHIFT, SW57 UPROW, SW58 PGDOWN, SW59 CRTL, SW6 #5, SW60 WIN, SW61 ALT, SW62 SPACE, SW63 ALT, SW64 FN, SW65 LEFTROW, SW66 DOWNROW, SW67 RIGHTROW, SW7 #6, SW8 #7, SW9 #8, U1 PRTR5V0U2X, U2 ATmega32U4-A, Y1 Crystal_GND24_Small

Commit message: Saving Progress on Part 3
Parts:
- moved D15 41.4 mm to (327.8, 76.4)
- moved F1 40.8 mm to (179.4, 70.9)
- moved D16 40.7 mm to (46.8, 95.4)
- moved D1 40.7 mm to (42.1, 76.4)
- moved R3 40.7 mm to (181.8, 68.5)
- moved R4 40.6 mm to (176.9, 68.5)
- moved SW43 40.6 mm to (291.3, 110.2)
- moved D14 40.6 mm to (299.4, 76.4)
- moved SW57 40.6 mm to (303.2, 129.2)
- moved SW66 40.6 mm to (303.2, 148.3)
- moved D39 40.6 mm to (208.9, 114.5)
- moved D40 40.6 mm to (228.0, 114.5)
- moved SW37 40.6 mm to (165.1, 110.2)
- moved SW39 40.6 mm to (203.2, 110.2)
- moved D11 40.6 mm to (232.7, 76.4)
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Routing:
- net row0: track 0.00 -> 291.7 mm
- net col4: track 0.00 -> 286.3 mm
- net row2: track 0.00 -> 283.9 mm
- net row4: track 0.00 -> 281.9 mm
- net row3: track 0.00 -> 281.0 mm
- net col0: track 0.00 -> 21.6 mm
- net Net-(D16-A): track 0.00 -> 13.6 mm
Other:
- outline, holes or cut-outs redrawn
