File: pcb/pcb.kicad_pcb (KiCad board)
At the start: 2 copper layers, 305 x 104.8 mm, 155 parts, among them J1 AVR-ISP-6, SW1 ESCAPE, SW10 #9, SW11 #0, SW12 -_, SW13 =+, SW14 BKSPC, SW15 DELETE, SW16 TAB, SW17 Q, SW18 W, SW19 E, SW2 #1, SW20 R, SW21 T, SW22 Y, SW23 U, SW24 I, SW25 O, SW26 P, SW27 [{, SW28 ]}, SW29 \|, SW3 #2, SW30 `~, SW31 CAP, SW32 A, SW33 D, SW34 S, SW35 F, SW36 G, SW37 H, SW38 J, SW39 K, SW4 #3, SW40 L, SW41 ;:, SW42 '", SW43 ENTER, SW44 PGUP, SW45 SHIFT, SW46 Z, SW47 X, SW48 C, SW49 V, SW5 #4, SW50 B, SW51 N, SW52 M, SW53 ,<, SW54 .>, SW55 /?, SW56 SHIFT, SW57 UPROW, SW58 PGDOWN, SW59 CRTL, SW6 #5, SW60 WIN, SW61 ALT, SW62 SPACE, SW63 ALT, SW64 FN, SW65 LEFTROW, SW66 DOWNROW, SW67 RIGHTROW, SW7 #6, SW8 #7, SW9 #8, U1 PRTR5V0U2X, U2 ATmega32U4-A, Y1 Crystal_GND24_Small

Commit message: Routing Finished
Parts:
- moved J1 63.7 mm to (217.8, 141.4)
- moved R6 36.5 mm to (184.7, 154.8)
- moved R5 31.5 mm to (215.3, 150.8), turned to 0 degrees
- moved C5 18.7 mm to (181.5, 141.3), turned to 180 degrees
- moved F1 7.22 mm to (175.4, 76.9), turned to -90 degrees
- moved C2 4.49 mm to (208.8, 149.2)
- moved C3 4.41 mm to (208.8, 146.8)
- moved C1 4.11 mm to (190.7, 136.5)
- moved C8 3.69 mm to (182.8, 138.3)
- moved U1 3.44 mm to (179.4, 72.2)
- moved R1 2.82 mm to (184.9, 133.5)
- moved r7 2.57 mm to (223.8, 149.0), turned to 0 degrees
- moved Y1 2.52 mm to (203.9, 148.2), turned to 90 degrees
- moved R2 2.06 mm to (188.1, 133.6)
- moved C4 1.61 mm to (181.9, 150.8)
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Connections:
- net Net-(U1-IO1) renamed DP
- net Net-(U1-IO2) renamed DN
- D16 pad 1: col4 -> row1
- D17 pad 1: col4 -> row1
- D18 pad 1: col4 -> row1
- D19 pad 1: col4 -> row1
- D20 pad 1: col4 -> row1
- D21 pad 1: col4 -> row1
- D22 pad 1: col4 -> row1
- D23 pad 1: col4 -> row1
- D24 pad 1: col4 -> row1
- D25 pad 1: col4 -> row1
- D26 pad 1: col4 -> row1
- D27 pad 1: col4 -> row1
- D28 pad 1: col4 -> row1
- D29 pad 1: col4 -> row1
- D30 pad 1: col4 -> row1
- U2 pad 36: col6 -> row4
- U2 pad 37: col5 -> col6
- U2 pad 38: col4 -> col5
- U2 pad 39: row4 -> row1
Routing:
- net row1: track 0.00 -> 367.0 mm, vias 0 -> 6
- net GND: track 0.00 -> 292.1 mm, vias 0 -> 7
- net row0: track 291.7 -> 531.2 mm, vias 0 -> 6
- net col14: track 0.00 -> 233.4 mm, vias 0 -> 1
- net col0: track 21.6 -> 243.8 mm, vias 0 -> 1
- net col1: track 0.00 -> 216.9 mm, vias 0 -> 1
- net +5V: track 0.00 -> 213.8 mm, vias 0 -> 6
- net col13: track 0.00 -> 212.8 mm, vias 0 -> 1
- net col12: track 0.00 -> 208.0 mm, vias 0 -> 2
- net col2: track 0.00 -> 184.6 mm, vias 0 -> 1
- net col11: track 0.00 -> 167.7 mm, vias 0 -> 2
- net col3: track 0.00 -> 154.6 mm, vias 0 -> 1
- net col4: track 286.3 -> 134.0 mm, vias 0 -> 1
- net col9: track 0.00 -> 149.3 mm, vias 0 -> 1
- net col10: track 0.00 -> 149.0 mm
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- added copper zone on B.Cu, net GND
- added copper zone on F.Cu, net GND
