File: pcb/pcb.kicad_pcb (KiCad board)
At the start: 2 copper layers, 305 x 104.8 mm, 155 parts, among them J1 AVR-ISP-6, SW1 ESCAPE, SW10 #9, SW11 #0, SW12 -_, SW13 =+, SW14 BKSPC, SW15 DELETE, SW16 TAB, SW17 Q, SW18 W, SW19 E, SW2 #1, SW20 R, SW21 T, SW22 Y, SW23 U, SW24 I, SW25 O, SW26 P, SW27 [{, SW28 ]}, SW29 \|, SW3 #2, SW30 `~, SW31 CAP, SW32 A, SW33 D, SW34 S, SW35 F, SW36 G, SW37 H, SW38 J, SW39 K, SW4 #3, SW40 L, SW41 ;:, SW42 '", SW43 ENTER, SW44 PGUP, SW45 SHIFT, SW46 Z, SW47 X, SW48 C, SW49 V, SW5 #4, SW50 B, SW51 N, SW52 M, SW53 ,<, SW54 .>, SW55 /?, SW56 SHIFT, SW57 UPROW, SW58 PGDOWN, SW59 CRTL, SW6 #5, SW60 WIN, SW61 ALT, SW62 SPACE, SW63 ALT, SW64 FN, SW65 LEFTROW, SW66 DOWNROW, SW67 RIGHTROW, SW7 #6, SW8 #7, SW9 #8, U1 PRTR5V0U2X, U2 ATmega32U4-A, Y1 Crystal_GND24_Small

Commit message: Via stitching finished
Routing:
- net GND: track 266.4 -> 258.9 mm, vias 9 -> 31
- net col8: track 146.0 -> 143.9 mm
- net row1: track 367.0 -> 366.0 mm
- net row2: track 342.5 -> 343.6 mm
